File: pcb/WorldCubeProtoV1/WorldCubeProtoV1.kicad_pcb (KiCad board)
At the start: 4 copper layers, 75.8 x 54.3 mm, 120 parts, among them J1 iCESugar-pro, J10 KD040WXFPD014, J11 KD040WXFPD014-C015C_CTP, J12 VC-ADV7611, J13 AudioJack3_SwitchTR, J14 Conn_01x02, J15 Conn_01x02, J16 Conn_01x02, J17 Conn_01x02, J18 Conn_01x02, J19 Conn_01x02, J2 KD040WXFPD014, J3 KD040WXFPD014-C015C_CTP, J4 KD040WXFPD014, J5 KD040WXFPD014-C015C_CTP, J6 KD040WXFPD014, J7 KD040WXFPD014-C015C_CTP, J8 KD040WXFPD014, J9 KD040WXFPD014-C015C_CTP, U1 TCA9548ARGER, U2 PCM1681, U3 TLV61047DDC, U4 TLC59108xPW, U5 PAM8406D, U6 PAM8406D, U7 PAM8406D

Commit message: New prototype PCB progress
Parts:
- added H1: MountingHole_Pad, MountingHole:MountingHole_3.2mm_M3_Pad, F.Cu at (-36.0, -36.0)
- added H2: MountingHole_Pad, MountingHole:MountingHole_3.2mm_M3_Pad, F.Cu at (-36.0, 36.0)
- added H3: MountingHole_Pad, MountingHole:MountingHole_3.2mm_M3_Pad, F.Cu at (10.0, 41.0)
- added H4: MountingHole_Pad, MountingHole:MountingHole_3.2mm_M3_Pad, F.Cu at (45.0, 14.0)
- added J20: 5V, Connector_JST:JST_XH_B2B-XH-A_1x02_P2.50mm_Vertical, F.Cu at (33.1, -42.5)
- C11, C12, C14, C16, C17, C2, C20, C24, C28, C43, C44, C45, C46, JP3, JP4, JP5, R23, R24, R25, R26: moved to B.Cu
- D2, D5, JP2, R4: moved to F.Cu
- U2: footprint Package_SO:HTSSOP-28-1EP_4.4x9.7mm_P0.65mm_EP3.4x9.5mm_Mask2.4x6.17mm_ThermalVias -> Package_SO:HTSSOP-28-1EP_4.4x9.7mm_P0.65mm_EP3.4x9.5mm_Mask2.4x6.17mm
- moved J13 313.9 mm to (6.95, -52.6), turned to -90 degrees
- moved R23 297.8 mm to (3.40, -45.2), turned to 90 degrees
- moved C43 297.1 mm to (1.90, -45.2), turned to 90 degrees
- moved R24 296.5 mm to (5.65, -44.5)
- moved C44 295.0 mm to (5.65, -46.0)
- moved R25 293.5 mm to (7.58, -42.0), turned to -90 degrees
- moved C45 293.0 mm to (6.08, -42.0), turned to -90 degrees
- moved R26 292.6 mm to (9.82, -42.8)
- moved C46 290.2 mm to (9.82, -41.3)
- moved R16 274.4 mm to (-12.0, -45.0), turned to 90 degrees
- moved R15 271.8 mm to (-11.2, -42.7)
- moved C36 271.0 mm to (-10.5, -45.0), turned to 90 degrees
- moved C35 269.3 mm to (-11.2, -41.2)
- moved FB5 267.2 mm to (-10.6, -52.5), turned to 90 degrees
- moved R14 263.7 mm to (-25.4, -45.0), turned to 90 degrees
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Connections:
- A1 pad 1: unconnected-(A1-GPIO0-Pad1) -> ADV7611_~{RST}
- A1 pad 10: unconnected-(A1-GPIO7-Pad10) -> LCD_~{RST}
- A1 pad 11: unconnected-(A1-GPIO8-Pad11) -> I2C_SDA
- A1 pad 12: unconnected-(A1-GPIO9-Pad12) -> I2C_SCL
- A1 pad 14: unconnected-(A1-GPIO10-Pad14) -> LCD_SCL
- A1 pad 15: unconnected-(A1-GPIO11-Pad15) -> LCD_SDA
- A1 pad 16: unconnected-(A1-GPIO12-Pad16) -> CTP_~{RST}
- A1 pad 17: unconnected-(A1-GPIO13-Pad17) -> CTP_INT
- A1 pad 19: unconnected-(A1-GPIO14-Pad19) -> CTP_SDA
- A1 pad 2: unconnected-(A1-GPIO1-Pad2) -> LCD1_~{CS}
- A1 pad 20: unconnected-(A1-GPIO15-Pad20) -> CTP_SCL
- A1 pad 21: unconnected-(A1-GPIO16-Pad21) -> DAC_SCK
- A1 pad 22: unconnected-(A1-GPIO17-Pad22) -> DAC_BCK
- A1 pad 24: unconnected-(A1-GPIO18-Pad24) -> DAC_LRCK
- A1 pad 25: unconnected-(A1-GPIO19-Pad25) -> DAC_DATA1
- A1 pad 26: unconnected-(A1-GPIO20-Pad26) -> DAC_DATA2
- A1 pad 27: unconnected-(A1-GPIO21-Pad27) -> DAC_DATA3
- A1 pad 29: unconnected-(A1-GPIO22-Pad29) -> DAC_DATA4
- A1 pad 31: unconnected-(A1-GPIO26_ADC0-Pad31) -> AMP_~{MUTE}
- A1 pad 32: unconnected-(A1-GPIO27_ADC1-Pad32) -> AMP_~{SHDN}
- A1 pad 4: unconnected-(A1-GPIO2-Pad4) -> LCD5_~{CS}
- A1 pad 5: unconnected-(A1-GPIO3-Pad5) -> LCD2_~{CS}
- A1 pad 6: unconnected-(A1-GPIO4-Pad6) -> LCD_DRV_EN
- A1 pad 7: unconnected-(A1-GPIO5-Pad7) -> LCD3_~{CS}
- A1 pad 9: unconnected-(A1-GPIO6-Pad9) -> LCD4_~{CS}
- J14 pad 1: /AudioAmp/-OUT_L -> /AudioAmp/+OUT_L
- J14 pad 2: /AudioAmp/+OUT_L -> /AudioAmp/-OUT_L
- J15 pad 1: /AudioAmp/-OUT_R -> /AudioAmp/+OUT_R
- J15 pad 2: /AudioAmp/+OUT_R -> /AudioAmp/-OUT_R
- J16 pad 1: /AudioAmp1/-OUT_L -> /AudioAmp1/+OUT_L
- J16 pad 2: /AudioAmp1/+OUT_L -> /AudioAmp1/-OUT_L
- J17 pad 1: /AudioAmp1/-OUT_R -> /AudioAmp1/+OUT_R
- J17 pad 2: /AudioAmp1/+OUT_R -> /AudioAmp1/-OUT_R
- J18 pad 1: /AudioAmp2/-OUT_L -> /AudioAmp2/+OUT_L
- J18 pad 2: /AudioAmp2/+OUT_L -> /AudioAmp2/-OUT_L
- J19 pad 1: /AudioAmp2/-OUT_R -> /AudioAmp2/+OUT_R
- J19 pad 2: /AudioAmp2/+OUT_R -> /AudioAmp2/-OUT_R
- R2 pad 1: I2C_SCL -> I2C_SDA
- R3 pad 1: I2C_SDA -> I2C_SCL
- RN1 pad 1: CTP1_SDA -> CTP4_SDA
- RN1 pad 2: CTP1_SCL -> CTP4_SCL
- RN1 pad 3: CTP2_SDA -> unconnected-(RN1-R3.1-Pad3)
- RN1 pad 4: CTP2_SCL -> unconnected-(RN1-R4.1-Pad4)
- RN2 pad 1: CTP3_SDA -> CTP5_SDA
- RN2 pad 2: CTP3_SCL -> CTP5_SCL
- RN2 pad 3: CTP4_SDA -> CTP1_SDA
- RN2 pad 4: CTP4_SCL -> CTP1_SCL
- RN3 pad 1: CTP5_SDA -> CTP2_SDA
- RN3 pad 2: CTP5_SCL -> CTP2_SCL
- RN3 pad 3: unconnected-(RN3-R3.1-Pad3) -> CTP3_SDA
- RN3 pad 4: unconnected-(RN3-R4.1-Pad4) -> CTP3_SCL
- RN3 pad 5: unconnected-(RN3-R4.2-Pad5) -> +3V3
- RN3 pad 6: unconnected-(RN3-R3.2-Pad6) -> +3V3
- U1 pad 1: CTP1_SDA -> unconnected-(U1-SD0-Pad1)
- U1 pad 10: CTP5_SDA -> CTP1_SDA
- U1 pad 11: CTP5_SCL -> CTP1_SCL
- U1 pad 12: unconnected-(U1-SD5-Pad12) -> CTP2_SDA
- U1 pad 13: unconnected-(U1-SC5-Pad13) -> CTP2_SCL
- U1 pad 14: unconnected-(U1-SD6-Pad14) -> CTP3_SDA
- U1 pad 15: unconnected-(U1-SC6-Pad15) -> CTP3_SCL
- U1 pad 2: CTP1_SCL -> unconnected-(U1-SC0-Pad2)
- U1 pad 25: unconnected-(U1-1EP-Pad25) -> GND
- U1 pad 3: CTP2_SDA -> unconnected-(U1-SD1-Pad3)
- U1 pad 4: CTP2_SCL -> unconnected-(U1-SC1-Pad4)
- U1 pad 5: CTP3_SDA -> CTP4_SDA
- U1 pad 6: CTP3_SCL -> CTP4_SCL
- U1 pad 7: CTP4_SDA -> CTP5_SDA
- U1 pad 8: CTP4_SCL -> CTP5_SCL
- U2 pad 19: /AudioAmp2/INL -> /AudioAmp2/INR
- U2 pad 20: /AudioAmp2/INR -> /AudioAmp2/INL
- U2 pad 21: /AudioAmp1/INL -> /AudioAmp1/INR
- U2 pad 22: /AudioAmp1/INR -> /AudioAmp1/INL
- U2 pad 26: /AudioAmp/INL -> /AudioAmp/INR
- U2 pad 27: /AudioAmp/INR -> /AudioAmp/INL
- U4 pad 10: LEDK4 -> LEDK1
- U4 pad 11: LEDK5 -> LEDK2
- U4 pad 6: LEDK1 -> LEDK3
- U4 pad 7: LEDK2 -> LEDK4
- U4 pad 9: LEDK3 -> LEDK5
Routing:
- net +3V3: track 1.31 -> 324.7 mm, vias 0 -> 15
- net +5V: track 4.41 -> 299.5 mm, vias 0 -> 13
- net LEDA: track 3.71 -> 194.2 mm, vias 0 -> 7
- net CTP_~{RST}: track 8.00 -> 192.5 mm, vias 0 -> 5
- net CTP_INT: track 0.00 -> 183.2 mm, vias 0 -> 6
- net GND: track 8.30 -> 161.2 mm, vias 0 -> 350
- net LCD_SCL: track 0.00 -> 149.6 mm, vias 0 -> 4
- net LCD_SDA: track 0.00 -> 149.2 mm, vias 0 -> 4
- net LCD_~{RST}: track 0.00 -> 138.3 mm, vias 0 -> 5
- net I2C_SCL: track 0.00 -> 123.3 mm, vias 0 -> 4
- net I2C_SDA: track 0.00 -> 115.8 mm, vias 0 -> 4
- net LCD4_~{CS}: track 0.00 -> 86.8 mm, vias 0 -> 2
- net CTP2_SCL: track 0.00 -> 84.5 mm, vias 0 -> 3
- net CTP2_SDA: track 0.00 -> 84.0 mm, vias 0 -> 3
- net LEDK1: track 0.00 -> 80.4 mm, vias 0 -> 2
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- added copper zone on In1.Cu, net GND
- added copper zone on In2.Cu, net GND
Other:
- board size 75.8 x 54.3 mm -> 95.2 x 112.5 mm
