File: pcb/WorldCubeProtoV1/WorldCubeProtoV1.kicad_sch (KiCad schematic)
At the start: 65 parts, among them J1 iCESugar-pro, J10 KD040WXFPD014, J11 KD040WXFPD014-C015C_CTP, J12 VC-ADV7611, J13 AudioJack3_SwitchTR, J14 Conn_01x02, J15 Conn_01x02, J16 Conn_01x02, J17 Conn_01x02, J18 Conn_01x02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

Commit message: New prototype PCB progress
Parts:
- added H1, H2, H3, H4: MountingHole_Pad, MountingHole:MountingHole_3.2mm_M3_Pad, symbol Mechanical:MountingHole_Pad
- U2: footprint Package_SO:HTSSOP-28-1EP_4.4x9.7mm_P0.65mm_EP3.4x9.5mm_Mask2.4x6.17mm_ThermalVias -> Package_SO:HTSSOP-28-1EP_4.4x9.7mm_P0.65mm_EP3.4x9.5mm_Mask2.4x6.17mm
Connections:
- net +3V3: now also RN3.5 (R4.2), RN3.6 (R3.2)
- net ADV7611_~{RST}: now also A1.1 (GPIO0)
- net AMP_~{MUTE}: now also A1.31 (GPIO26_ADC0)
- net AMP_~{SHDN}: now also A1.32 (GPIO27_ADC1)
- net AudioAmp/+OUT_L: now also J14.1 (Pin_1); no longer J14.2 (Pin_2)
- net AudioAmp/+OUT_R: now also J15.1 (Pin_1); no longer J15.2 (Pin_2)
- net AudioAmp/-OUT_L: now also J14.2 (Pin_2); no longer J14.1 (Pin_1)
- net AudioAmp/-OUT_R: now also J15.2 (Pin_2); no longer J15.1 (Pin_1)
- net AudioAmp/INL: now also U2.27 (V_{out}1); no longer U2.26 (V_{out}2)
- net AudioAmp/INR: now also U2.26 (V_{out}2); no longer U2.27 (V_{out}1)
- net AudioAmp1/+OUT_L: now also J16.1 (Pin_1); no longer J16.2 (Pin_2)
- net AudioAmp1/+OUT_R: now also J17.1 (Pin_1); no longer J17.2 (Pin_2)
- net AudioAmp1/-OUT_L: now also J16.2 (Pin_2); no longer J16.1 (Pin_1)
- net AudioAmp1/-OUT_R: now also J17.2 (Pin_2); no longer J17.1 (Pin_1)
- net AudioAmp1/INL: now also U2.22 (V_{out}3); no longer U2.21 (V_{out}4)
- net AudioAmp1/INR: now also U2.21 (V_{out}4); no longer U2.22 (V_{out}3)
- net AudioAmp2/+OUT_L: now also J18.1 (Pin_1); no longer J18.2 (Pin_2)
- net AudioAmp2/+OUT_R: now also J19.1 (Pin_1); no longer J19.2 (Pin_2)
- net AudioAmp2/-OUT_L: now also J18.2 (Pin_2); no longer J18.1 (Pin_1)
- net AudioAmp2/-OUT_R: now also J19.2 (Pin_2); no longer J19.1 (Pin_1)
- net AudioAmp2/INL: now also U2.20 (V_{out}5); no longer U2.19 (V_{out}6)
- net AudioAmp2/INR: now also U2.19 (V_{out}6); no longer U2.20 (V_{out}5)
- net CTP1_SCL: now also RN2.4 (R4.1), U1.11 (SC4); no longer RN1.2 (R2.1), U1.2 (SC0)
- net CTP1_SDA: now also RN2.3 (R3.1), U1.10 (SD4); no longer RN1.1 (R1.1), U1.1 (SD0)
- net CTP2_SCL: now also RN3.2 (R2.1), U1.13 (SC5); no longer RN1.4 (R4.1), U1.4 (SC1)
- net CTP2_SDA: now also RN3.1 (R1.1), U1.12 (SD5); no longer RN1.3 (R3.1), U1.3 (SD1)
- net CTP3_SCL: now also RN3.4 (R4.1), U1.15 (SC6); no longer RN2.2 (R2.1), U1.6 (SC2)
- net CTP3_SDA: now also RN3.3 (R3.1), U1.14 (SD6); no longer RN2.1 (R1.1), U1.5 (SD2)
- net CTP4_SCL: now also RN1.2 (R2.1), U1.6 (SC2); no longer RN2.4 (R4.1), U1.8 (SC3)
- net CTP4_SDA: now also RN1.1 (R1.1), U1.5 (SD2); no longer RN2.3 (R3.1), U1.7 (SD3)
- net CTP5_SCL: now also RN2.2 (R2.1), U1.8 (SC3); no longer RN3.2 (R2.1), U1.11 (SC4)
- net CTP5_SDA: now also RN2.1 (R1.1), U1.7 (SD3); no longer RN3.1 (R1.1), U1.10 (SD4)
- net CTP_INT: now also A1.17 (GPIO13)
- net CTP_SCL: now also A1.20 (GPIO15)
- net CTP_SDA: now also A1.19 (GPIO14)
- net CTP_~{RST}: now also A1.16 (GPIO12)
- net DAC_BCK: now also A1.22 (GPIO17)
- net DAC_DATA1: now also A1.25 (GPIO19)
- net DAC_DATA2: now also A1.26 (GPIO20)
- net DAC_DATA3: now also A1.27 (GPIO21)
- net DAC_DATA4: now also A1.29 (GPIO22)
- net DAC_LRCK: now also A1.24 (GPIO18)
- net DAC_SCK: now also A1.21 (GPIO16)
- net GND: now also U1.25 (EP), H1.1, H2.1, H3.1, H4.1
- net I2C_SCL: now also A1.12 (GPIO9), R3.1; no longer R2.1
- net I2C_SDA: now also A1.11 (GPIO8), R2.1; no longer R3.1
- net LCD1_~{CS}: now also A1.2 (GPIO1)
- net LCD2_~{CS}: now also A1.5 (GPIO3)
- net LCD3_~{CS}: now also A1.7 (GPIO5)
- net LCD4_~{CS}: now also A1.9 (GPIO6)
- net LCD5_~{CS}: now also A1.4 (GPIO2)
- net LCD_DRV_EN: now also A1.6 (GPIO4)
- net LCD_SCL: now also A1.14 (GPIO10)
- net LCD_SDA: now also A1.15 (GPIO11)
- net LCD_~{RST}: now also A1.10 (GPIO7)
- net LEDK1: now also U4.10 (~{OUT3}); no longer U4.6 (~{OUT0})
- net LEDK2: now also U4.11 (~{OUT4}); no longer U4.7 (~{OUT1})
- net LEDK3: now also U4.6 (~{OUT0}); no longer U4.9 (~{OUT2})
- net LEDK4: now also U4.7 (~{OUT1}); no longer U4.10 (~{OUT3})
- net LEDK5: now also U4.9 (~{OUT2}); no longer U4.11 (~{OUT4})
- no-connect marks 153 -> 149
Other:
- moved on the sheet: A1
